File: asic/e-class-aardonyx/board/Board_Design/soc.sch (KiCad schematic (older format))
At the start: 111 parts, among them SW3 SW_DIP_x03, U15 SKT32E

Commit message: Updating layout after back annotation
Parts:
- renumbered C88 to C10, C64 to C13, C65 to C19, C82 to C2, C89 to C20, C87 to C24, C86 to C25, C79 to C3, C84 to C30, C63 to C31, C68 to C32, C83 to C33, C81 to C34, C78 to C37, C80 to C39, C66 to C41, C71 to C42, C75 to C48, C76 to C5, C74 to C51, C69 to C52, C77 to C53, C72 to C54, C73 to C6, C90 to C7, C70 to C8, C67 to C9, D8 to D1, D7 to D2, D6 to D3, R82 to R10, R83 to R11, R78 to R12, R80 to R13, R87 to R14, R86 to R15, R85 to R16, R84 to R17, R81 to R19, R99 to R20, R79 to R21, R100 to R22, R88 to R23, R89 to R24, R101 to R25, R102 to R26, R103 to R27, R44 to R3, R104 to R30, R105 to R31, R106 to R33, R107 to R34, R108 to R37, R109 to R38, R43 to R4, R110 to R40, R111 to R41, R62 to R42, R61 to R44, R64 to R47, R112 to R48, R113 to R49, R42 to R5, R63 to R52, R60 to R54, R59 to R55, R58 to R56, R114 to R57, R116 to R58, R115 to R59, R57 to R61, R117 to R62, R124 to R64, R122 to R65, R120 to R66, R118 to R67, R125 to R68, R123 to R69, R96 to R7, R121 to R70, R126 to R71, R131 to R72, R77 to R73, R127 to R74, R119 to R75, R75 to R77, R65 to R78, R66 to R79, R97 to R8, R128 to R80, R95 to R81, R93 to R82, R92 to R83, R90 to R84, R94 to R85, R91 to R86, R74 to R87, R73 to R88, R72 to R89, R98 to R9, R71 to R90, R70 to R91, R69 to R92, R68 to R93, R67 to R94, R129 to R95, R132 to R96, R130 to R97, SW3 to SW2, U15 to U2
