File: asic/e-class-aardonyx/board/Board_Design/Aardonyx_Socket/Aardonyx.sch (KiCad schematic (older format))
At the start: 9 parts

Commit message: updated soc back annotation
Parts:
- added H8: MountingHole, MountingHole:MountingHole_3.2mm_M3, symbol Mechanical:MountingHole
Changed lines of the file:
@@
 Text Label 7350 4950 0    50   ~ 0
 RESET
+$Comp
+L Mechanical:MountingHole H8
+U 1 1 5F3B4871
+P 3300 7250
+F 0 "H8" H 3400 7296 50  0000 L CNN
+F 1 "MountingHole" H 3400 7205 50  0000 L CNN
+F 2 "MountingHole:MountingHole_3.2mm_M3" H 3300 7250 50  0001 C CNN
+F 3 "~" H 3300 7250 50  0001 C CNN
+	1    3300 7250
+	1    0    0    -1
+$EndComp
 $EndSCHEMATC
