File: asic/e-class-aardonyx/board/Board_Design/Aardonyx_Socket/Aardonyx.kicad_pcb (KiCad board)
At the start: 4 copper layers, 329 parts, among them J1 Conn_1x4, J10 Conn_1x3_M, J11 Conn_1x8, J12 Conn_1x3_M, J13 USB_B_6PIN, J14 Conn_1x4, J15 Conn_1x3_M, J16 USB_OTG, J17 Conn_1x8, J18 Conn_1x3_M, J19 Conn_1x3_M, J2 Conn_1x6, J3 Conn_1x10_F, J4 Conn_1x8_F, J5 Conn_1x8_F, J6 Conn_1x6_F, J7 Conn_1x3_M, J8 PJ-202H PWRJACK, J9 Conn_1x6, Q1 FDN339AN, SW1 FSM2JSMAATR, SW2 SW_DIP_x03, SW3 SW_SPST, U1 LSF0108PWR, U10 ADM1186, U11 FT2232H, U12 TPS7A7002DDAR, U13 TPS54627DDAR, U14 93LC56BT-I_OT, U15 TPS7A7002DDAR, U2 SKT32E, U3 IS42S32160F-TSOP2, U4 LSF0108PWR, U5 CDCE913PW, U6 ADC128S102CIMTX/NOPB, U7 74AUP1G09GW, U8 IS25LP256x-xM, U9 CAT24M01WI-GT3, Y1 27MHz, Y2 12MHz

Commit message: updated soc back annotation
Parts:
- added H8: MountingHole, MountingHole:MountingHole_3.2mm_M3, F.Cu at (278.9, 16.9)
- FB3, FB7: value 47E,FB,0402 -> 47E,FB,0603; footprint Inductor_SMD:L_0402_1005Metric -> Inductor_SMD:L_0603_1608Metric
- U9: footprint Package_SO:SOIC-8_3.9x4.9mm_P1.27mm -> Package_SO:SOIC-8_5.23x5.23mm_P1.27mm
- moved H6 4.79 mm to (48.4, 156.7)
- moved C58 1.58 mm to (121.9, 144.6)
- moved U9 0.80 mm to (128.9, 143.3)
- moved H3 0.10 mm to (49.1, 17.7)
Routing:
- net GND: track 412.9 -> 430.2 mm, vias 161 -> 160
- net V3P3: track 252.3 -> 256.2 mm
- net /arduino_header/I2C0_SCL: track 91.5 -> 90.9 mm
- net VAC: vias 1 -> 2
Other:
- board text added: "I2C0"
- board text added: "RX"
- board text added: "TX"
- board text added: "UART0"

Commit message: Back annotation
Parts:
- renumbered C44 to C1, C3 to C10, C29 to C11, C5 to C12, C6 to C13, C8 to C14, C9 to C15, C13 to C16, C16 to C17, C17 to C18, C47 to C2, C25 to C21, C24 to C22, C46 to C23, C31 to C24, C30 to C25, C23 to C26, C32 to C27, C34 to C28, C27 to C29, C1 to C3, C28 to C30, C33 to C31, C49 to C32, C41 to C33, C37 to C34, C38 to C35, C50 to C36, C42 to C37, C26 to C38, C12 to C39, C7 to C4, C39 to C40, C48 to C41, C14 to C42, C36 to C43, C35 to C44, C54 to C46, C21 to C47, C40 to C48, C52 to C49, C4 to C5, C15 to C50, C43 to C51, C18 to C52, C51 to C53, C53 to C54, C95 to C55, C55 to C56, C56 to C57, C60 to C58, C61 to C59, C10 to C6, C62 to C60, C63 to C61, C64 to C62, C65 to C63, C66 to C64, C67 to C65, C68 to C66, C69 to C67, C59 to C68, C71 to C69, C11 to C7, C81 to C70, C70 to C71, C77 to C74, C58 to C75, C57 to C76, C80 to C77, C82 to C78, C89 to C79, C22 to C8, C90 to C80, C92 to C81, C93 to C82, C74 to C83, C76 to C84, C78 to C85, C79 to C86, C75 to C87, C91 to C89, C2 to C9, C97 to C90, C83 to C91, C84 to C92, C85 to C93, C86 to C94, C87 to C95, C94 to C96, C96 to C97, FB7 to FB1, FB5 to FB2, FB1 to FB3, FB6 to FB4, FB3 to FB5, FB2 to FB6, FB4 to FB7, J2 to J1, J8 to J10, J16 to J12, J12 to J13, J13 to J14, J14 to J16, J3 to J2, J4 to J3, J5 to J4, J6 to J5, J1 to J6, J9 to J8, J10 to J9, R3 to R1, R60 to R10, R79 to R100, R78 to R101, R106 to R102, R107 to R103, R108 to R104, R109 to R105, R116 to R106, R117 to R107, R118 to R108, R119 to R109, R63 to R11, R127 to R110, R128 to R111, R122 to R112, R123 to R113, R124 to R114, R81 to R115, R82 to R116, R85 to R117, R84 to R118, R83 to R119, R23 to R12, R86 to R120, R131 to R121, R133 to R122, R137 to R123, R125 to R124, R126 to R125, R134 to R126, R135 to R127, R104 to R128, R105 to R129, R12 to R13, R98 to R130, R103 to R131, R120 to R132, R121 to R133, R142 to R134, R143 to R135, R138 to R136, R145 to R137, R147 to R138, R148 to R139, R24 to R14, R129 to R140, R130 to R141, R132 to R142, R136 to R143, R139 to R144, R140 to R145, R141 to R146, R144 to R147, R150 to R148, R151 to R149, R21 to R15, R153 to R150, R152 to R151, R146 to R152, R149 to R153, R14 to R16, R15 to R17, R16 to R18, R17 to R19, R4 to R2, R7 to R20, R72 to R21, R8 to R22, R9 to R23, R80 to R24, R18 to R25, R95 to R26, R96 to R27, R97 to R28, R19 to R29, R5 to R3, R10 to R30, R11 to R31, R20 to R32, R13 to R33, R22 to R34, R25 to R35, R26 to R36, R27 to R37, R30 to R38, R43 to R39, R45 to R4, R31 to R40, R33 to R41, R34 to R42, R37 to R43, R38 to R44, R28 to R45, R29 to R46, R40 to R47, R41 to R48, R32 to R49, R46 to R5, R35 to R50, R48 to R51, R36 to R52, R42 to R53, R49 to R54, R44 to R55, R57 to R56, R39 to R57, R47 to R58, R52 to R59, R50 to R6, R59 to R60, R58 to R61, R54 to R62, R55 to R63, R61 to R64, R56 to R65, R62 to R66, R1 to R68, R2 to R69, R51 to R7, R75 to R70, R74 to R71, R71 to R72, R68 to R73, R64 to R74, R70 to R75, R66 to R76, R99 to R77, R100 to R78, R101 to R79, R53 to R8, R102 to R80, R110 to R81, R111 to R82, R112 to R83, R113 to R84, R114 to R85, R115 to R86, R65 to R87, R69 to R88, R77 to R89, R6 to R9, R73 to R90, R76 to R91, R87 to R92, R88 to R93, R89 to R94, R90 to R95, R91 to R96, R92 to R97, R93 to R98, R94 to R99, U2 to U1, U11 to U10, U9 to U11, U8 to U12, U15 to U14, U14 to U15, U1 to U2, U7 to U3, U6 to U5, U5 to U6, U3 to U7, U10 to U8, U12 to U9
Routing:
- net GND: track 430.2 -> 432.2 mm, vias 160 -> 158
- net /ftdi/D-: track 41.4 -> 40.8 mm
- net /ftdi/D+: track 41.4 -> 40.9 mm
- net V3P3: vias 65 -> 67
- net Net-(C69-Pad1): vias 4 -> 3
- added copper zone on B.Cu, net V3P3
- removed copper zone on In2.Cu, net Net-(C69-Pad1)
Other:
- board outline added: 240.5 x 150.9 mm
- rule trace_min: 0 -> 0.2032

Commit message: updated soc drc error
Parts:
- moved H4 2.52 mm to (279.1, 157.6)
- moved H3 1.11 mm to (48.6, 16.7)
- moved H6 0.89 mm to (48.6, 157.6)
- moved H8 0.27 mm to (279.1, 16.7)

Commit message: Final layout files
Parts:
- moved H8 0.30 mm to (278.8, 16.6)
- moved H4 0.27 mm to (278.8, 157.6)
Routing:
- net V1P8: track 437.6 -> 436.6 mm
- net /soc/TD0: track 123.9 -> 123.3 mm
- net /ftdi/TMS: track 140.0 -> 139.3 mm
- net /ftdi/TDI: track 134.5 -> 133.8 mm
- net VAC: track 106.5 -> 107.1 mm
- net Net-(C80-Pad2): vias 0 -> 3
- added copper zone on B.Cu, net Net-(C80-Pad2)
- added copper zone on In2.Cu, net Net-(C80-Pad2)
- added copper zone on B.Cu, net V1P8
- added copper zone on In2.Cu, net VBUS
Other:
- board size 240.5 x 150.9 mm -> 240.3 x 150.9 mm
- board text added: "Ardonyx MS Version 1.0 IIT MADRAS"
- board text added: "L1"
- board text added: "L4"
